File: v1.10/Lotus58_BLE.kicad_sch (KiCad schematic)
At the start: 160 parts, among them J1 USB_C_Receptacle_USB2.0, J2 BATT, J3 ProgConn, Q1 2N7002, Q2 2N7002, Q3 AO3401A, SW1 SW_Push, SW10 SW_Push, SW11 SW_Push, SW12 SW_Push, SW13 SW_Push, SW14 SW_Push, SW15 SW_Push, SW16 SW_Push, SW17 SW_Push, SW18 SW_Push, SW19 SW_Push, SW2 SW_Push, SW20 SW_Push, SW21 SW_Push, SW22 SW_Push, SW23 SW_Push, SW24 SW_Push, SW25 SW_Push, SW26 SW_Push, SW27 SW_Push, SW28 SW_Push, SW29 SW_Push, SW3 SW_Push, SW4 SW_Push, SW5 SW_Push, SW6 SW_Push, SW7 SW_Push, SW8 SW_Push, SW9 SW_Push, U1 BQ24075RGT, U2 E73-2G4M08S1C_test, U3 SRV05-4, U4 SN74LV1T34DBV, U7 E73-2G4M08S1C_test, Y1 XC32M4-32.768-F12NJDTL

Commit message: v1.1.0
Parts:
- added D+12: D, Diode_SMD:D_SOD-323, symbol Device:D
- J3: footprint Connector_PinHeader_1.27mm:PinHeader_1x05_P1.27mm_Vertical -> Connector_PinHeader_2.00mm:PinHeader_1x04_P2.00mm_Vertical; symbol Connector_Generic:Conn_01x05 -> Connector_Generic:Conn_01x04
- PWR_SW1, RES1: now fitted
- PWR_SW2, RES2: now left out of the parts list
Connections:
- net +3.3V: now also J3.4 (Pin_4); no longer J3.5 (Pin_5)
- net EncA: now also U2.1 (P1.11), U7.1 (P1.11); no longer U2.2 (P1.10), U7.2 (P1.10)
- net Pin0: now also D+12.2 (A)
- net RESET: no longer J3.4 (Pin_4)
- net ZMK_LED: now also U2.2 (P1.10), U7.2 (P1.10); no longer U2.1 (P1.11), U7.1 (P1.11)
- net at D+6.1 (K), SW26.2, SW27.2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: now also D+12.1 (K)
Other:
- note added: "Added missind diode. Should fix crystal, VCCH"
